File: kicad/base/base.sch (KiCad schematic (older format))
At the start: 23 parts, among them J1 Conn_01x05, Q1 MMBT3904, Q2 MMBT3904, Q3 MMBT3904, SW2 SW_SPST_LED_RGB, U1 Seeeduiono_Xiao, U2 NC7SB3257P6X, U3 AS5600

Commit message: something
Parts:
- C1: LCSC (none) -> C49678
- Q1, Q2, Q3: LCSC (none) -> C20526
- R1, R10, R8, R9: LCSC (none) -> C27834
- R2, R3, R4: LCSC (none) -> C17414
- R5: value 65R -> 68R; LCSC (none) -> C17802
- R6, R7: LCSC (none) -> C17415
Changed lines of the file:
@@
 F 2 "Resistor_SMD:R_0805_2012Metric" V 7380 5000 50  0001 C CNN
 F 3 "~" H 7450 5000 50  0001 C CNN
+F 4 "C17414" H 7450 5000 50  0001 C CNN "LCSC"
 	1    7450 5000
 	1    0    0    -1
@@
 F 2 "Resistor_SMD:R_0805_2012Metric" V 6030 5000 50  0001 C CNN
 F 3 "~" H 6100 5000 50  0001 C CNN
+F 4 "C27834" H 6100 5000 50  0001 C CNN "LCSC"
 	1    6100 5000
 	1    0    0    -1
@@
 F 2 "Resistor_SMD:R_0805_2012Metric" V 6480 5000 50  0001 C CNN
 F 3 "~" H 6550 5000 50  0001 C CNN
+F 4 "C17414" H 6550 5000 50  0001 C CNN "LCSC"
 	1    6550 5000
 	1    0    0    -1
@@
 F 2 "Resistor_SMD:R_0805_2012Metric" V 6930 5000 50  0001 C CNN
 F 3 "~" H 7000 5000 50  0001 C CNN
+F 4 "C17414" H 7000 5000 50  0001 C CNN "LCSC"
 	1    7000 5000
 	1    0    0    -1
@@
 F 2 "Capacitor_SMD:C_0805_2012Metric" H 6700 3600 50  0001 C CNN
 F 3 "~" H 6700 3600 50  0001 C CNN
+F 4 "C49678" H 6700 3600 50  0001 C CNN "LCSC"
 	1    6700 3600
 	1    0    0    -1
@@
 P 3150 1950
 F 0 "R5" V 3150 1950 50  0000 C CNN
-F 1 "65R" V 3250 1950 50  0000 C CNN
+F 1 "68R" V 3250 1950 50  0000 C CNN
 F 2 "Resistor_SMD:R_0805_2012Metric" V 3080 1950 50  0001 C CNN
 F 3 "~" H 3150 1950 50  0001 C CNN
+F 4 "C17802" V 3150 1950 50  0001 C CNN "LCSC"
 	1    3150 1950
 	0    1    1    0
@@
 F 2 "Resistor_SMD:R_0805_2012Metric" V 3080 2350 50  0001 C CNN
 F 3 "~" H 3150 2350 50  0001 C CNN
+F 4 "C17415" V 3150 2350 50  0001 C CNN "LCSC"
 	1    3150 2350
 	0    1    1    0
@@
 F 2 "Resistor_SMD:R_0805_2012Metric" V 3080 2150 50  0001 C CNN
 F 3 "~" H 3150 2150 50  0001 C CNN
+F 4 "C17415" V 3150 2150 50  0001 C CNN "LCSC"
 	1    3150 2150
 	0    1    1    0
@@
 F 2 "Package_TO_SOT_SMD:SOT-23" H 3550 4875 50  0001 L CIN
 F 3 "https://www.fairchildsemi.com/datasheets/2N/2N3904.pdf" H 3350 4950 50  0001 L CNN
+F 4 "C20526" H 3350 4950 50  0001 C CNN "LCSC"
 	1    3350 4950
 	1    0    0    -1
@@
 F 2 "Resistor_SMD:R_0805_2012Metric" V 2930 4950 50  0001 C CNN
 F 3 "~" H 3000 4950 50  0001 C CNN
+F 4 "C27834" V 3000 4950 50  0001 C CNN "LCSC"
 	1    3000 4950
 	0    1    1    0
@@
 F 2 "Package_TO_SOT_SMD:SOT-23" H 5150 5275 50  0001 L CIN
 F 3 "https://www.fairchildsemi.com/datasheets/2N/2N3904.pdf" H 4950 5350 50  0001 L CNN
+F 4 "C20526" H 4950 5350 50  0001 C CNN "LCSC"
 	1    4950 5350
 	1    0    0    -1
@@
 F 2 "Resistor_SMD:R_0805_2012Metric" V 4530 5350 50  0001 C CNN
 F 3 "~" H 4600 5350 50  0001 C CNN
+F 4 "C27834" V 4600 5350 50  0001 C CNN "LCSC"
 	1    4600 5350
 	0    1    1    0
@@
 F 2 "Package_TO_SOT_SMD:SOT-23" H 4750 4575 50  0001 L CIN
 F 3 "https://www.fairchildsemi.com/datasheets/2N/2N3904.pdf" H 4550 4650 50  0001 L CNN
+F 4 "C20526" H 4550 4650 50  0001 C CNN "LCSC"
 	1    4550 4650
 	1    0    0    -1
@@
 F 2 "Resistor_SMD:R_0805_2012Metric" V 4130 4650 50  0001 C CNN
 F 3 "~" H 4200 4650 50  0001 C CNN
+F 4 "C27834" V 4200 4650 50  0001 C CNN "LCSC"
 	1    4200 4650
 	0    1    1    0
